File: src/Design/_001_Get_start/Get_Start/Get_Start.kicad_sch (KiCad schematic)
At the start: 0 parts

Commit message: :link: hotkeys in schematic mode
Parts:
- added D1, D2, D3, D4, D5, D6: LED, symbol Device:LED
- added SW1: SW_SPST, symbol Switch:SW_SPST
Connections:
- new net label_A: SW1.1 (A), SW1.2 (B)
Other:
- note added: "A - get symbol"
- note added: "Click + G - drag object and wire"
- note added: "Click + M - drag object only"
- note added: "L - Label_A connect pin 1 and 2 of switch, short circuit reach when push switch on"
- note added: "R -Rotate"
- note added: "X - Mirror horizontal"
- note added: "Y - Mirror vertical"
- company: (none) -> HOME
- title: (none) -> GETTING STARTED SCHEMATIC
