File: src/Design/_001_Get_start/Get_Start/Get_Start.kicad_pcb (KiCad board)
At the start: 4 copper layers, 9.1 x 2 mm, 1 part, among them SW2 100 abc

Commit message: :yawning_face: done getting start with KiCad 9
Parts:
- moved SW2 102.4 mm to (165.1, 114.3)
Other:
- board size 9.1 x 2 mm -> 127 x 76.2 mm
Changed lines of the file:
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@@
 	(footprint "Simple_test_library:First component"
 		(layer "F.Cu")
-		(at 76.13 63.66)
+		(at 165.1 114.3)
 		(descr "Test component")
 		(property "Reference" "SW2"
@@
 		(embedded_fonts no)
 	)
+	(gr_rect
+		(start 101.6 76.2)
+		(end 228.6 152.4)
+		(stroke
+			(width 0.05)
+			(type default)
+		)
+		(fill no)
+		(layer "Edge.Cuts")
+	)
 	(embedded_fonts no)
